File: Projects/IR Hub for RPi v3.0/RasPi-BplusHAT.sch (EAGLE design)
At the start: 42 parts, among them SW1 SPST_TACT-KMR2, SW2 SPST_TACT-KMR2, SW3 SPST_TACT-KMR2, T1 2N4401, T2 2N4401, T3 2N4401, T4 2N4401, T5 2N4401, U1 CLVC1G32MDCKREPG4

Commit message: removed Watchdog
... as there is a hardware watchdog on Raspberry Pi, and a good
watchdog daemon  framework for health monitoring
Parts:
- removed R16, R17, R18: 1K, adafruit:R-US_R0805
- removed STM6823: STM6823STM6823, varshneya:STM6823STM6823
- removed T5: 2N4401, transistor-neu-to92:MMBT4401LT1-NPN-SOT23-BEC
- removed U1: CLVC1G32MDCKREPG4, Texas Instruments_By_element14_Batch_1:CLVC1G32MDCKREPG4
Connections:
- removed net N$12: C3.1, R14.1, STM6823.^MR, SW3.S, SW3.S1
- removed net N$15: R16.2, T5.C, U1.A
- removed net N$20: R17.2, R18.1, T5.B
- removed net N$9: STM6823.^RST, U1.B
- net +3V3: no longer R16.1, STM6823.VCC, U1.VCC
- net GND: no longer R18.2, STM6823.VSS, T5.E, U1.GND
- net GPIO21: no longer STM6823.WDI
- net GPIO26: no longer R17.1
- net RST: now also C3.1, R14.1, SW3.S, SW3.S1; no longer U1.Y
Other:
- note added: "Manual Reset"
- note added: "Need to add Schmitt triggers for debouncing these push buttons"
- note removed: "Replace this OR gate with a dual Schmitt trigger -- Much cheaper!!"
- note removed: "Reset/Watchdog"
- note removed: "WATCHDOG"
- note removed: "WD_ENABLE"
- moved on the sheet: C3, R14, SW3

Commit message: Cleaned up the board layout
... with name and blog URL added; added a smoothening aspect in the
circuit for the RESET push button.
Parts:
- added R15: 100K, adafruit:R-US_R0805
- R14: value 10K -> 1M
- renumbered LED8-IR-RVC to LED8-IR-RCV, LED9-HLTH to LED9-WARN
Connections:
- new net N$1: R15.2, SW3.S, SW3.S1
- net RST: now also R15.1; no longer SW3.S, SW3.S1
Other:
- moved on the sheet: C1, C2, C3, R12, R13, R14, SW1, SW2, SW3
